Commit message: update camera system part

File: assets/robot_car/urdf/robot_car.urdf (robot description, URDF)
Before this commit: robot ackermann_robot, 8 links, 7 joints
Links:
- added link camera_link; visual mesh filename=file:///home/eun/personal_project/humanoid_digital_twin/ass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
- added link pitch_base; visual mesh filename=file:///home/eun/personal_project/humanoid_digital_twin/ass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
- added link yaw_base; visual mesh filename=file:///home/eun/personal_project/humanoid_digital_twin/ass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
- link base_link: mass 2.0 -> None; geometry collision box size=0.225 0.14 0.13; visual mesh filename=file:///home/eun/personal_project/humanoid_digital_twin/ass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
- link front_left_steer: geometry 
- link front_right_steer: geometry 
Joints:
- removed joint rear_left_joint
- removed joint rear_right_joint
- added joint camera_joint: type fixed, parent pitch_base, child camera_link, origin xyz=0 0 0.005 rpy=0 0 0
- added joint pitch_joint: type revolute, parent yaw_base, child pitch_base, origin xyz=0 0 0.057646 rpy=0 0 0, axis 0 1 0, limit lower=-1.57 upper=1.57 effort=1.0 velocity=1.0
- added joint rear_left_wheel_joint: type continuous, parent base_link, child rear_left_wheel, origin xyz=-0.08 0.085 0.0335 rpy=0 0 0, axis 0 1 0
- added joint rear_right_wheel_joint: type continuous, parent base_link, child rear_right_wheel, origin xyz=-0.08 -0.085 0.0335 rpy=0 0 0, axis 0 1 0
- added joint yaw_joint: type revolute, parent base_link, child yaw_base, origin xyz=-0.076562 -0.000014 0.128658 rpy=0 0 0, axis 0 0 1, limit lower=-3.14 upper=3.14 effort=1.0 velocity=1.0
- joint base_joint: origin xyz=0 0 0 rpy=0 0 0 -> (none)
- joint front_left_steer_joint: limit lower=-0.52 upper=0.52 effort=1.0 velocity=1.0 -> lower=-0.52 upper=0.52 effort=10.0 velocity=1.0; origin xyz=0.07 0.0825 0.0335 rpy=0 0 0 -> xyz=0.08 0.085 0.0335 rpy=0 0 0
- joint front_right_steer_joint: limit lower=-0.52 upper=0.52 effort=1.0 velocity=1.0 -> lower=-0.52 upper=0.52 effort=10.0 velocity=1.0; origin xyz=0.07 -0.0825 0.0335 rpy=0 0 0 -> xyz=0.08 -0.085 0.0335 rpy=0 0 0

Commit message: add nav2 and slam for frontier and control

File: assets/robot_car/urdf/robot_car.urdf (robot description, URDF)
Before this commit: robot ackermann_gimbal_robot, 11 links, 10 joints
Links:
- added link lidar_frame
Joints:
- added joint lidar_joint: type fixed, parent base_link, child lidar_frame, origin xyz=-0.076562 -0.000014 0.128658 rpy=0 0 0
